File: Eagle Files/kinesisBLE V3.brd (EAGLE design)
At the start: 122 x 86 mm, 28 parts, among them X1 JST-XH-02-PIN-ROUND-PAD, X2 JST-XH-02-PIN-ROUND-PAD, X3 JST-XH-02-PIN-ROUND-PAD

Commit message: v3 board files
Parts:
- moved U$2 3.00 mm to (16.0, 74.0)
- moved U$3 3.00 mm to (106.0, 74.0)
- moved U$6 2.00 mm to (102.0, 8.00)
- moved U$7 2.00 mm to (20.0, 8.00)
Routing:
- net COL-O: track 154.8 -> 159.0 mm
- net ROW-7: track 129.0 -> 125.0 mm
- net COL-N: track 153.3 -> 157.1 mm
- net COL-M: track 119.8 -> 123.0 mm
- net ROW-5: track 194.9 -> 197.9 mm
- net ROW-4: track 167.8 -> 170.8 mm
- net NUM: track 215.9 -> 218.4 mm
- net COL-J: track 164.4 -> 166.4 mm
- net SCR: track 250.2 -> 252.1 mm
- net COL-F: track 67.7 -> 69.7 mm
- net CAPS: track 203.3 -> 205.3 mm
- net ROW-3: track 171.1 -> 172.7 mm
- net ROW-1: track 161.2 -> 162.7 mm
- net ROW-2: track 167.2 -> 168.6 mm
- net COL-I: track 156.9 -> 155.7 mm
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